File: Hardware/Variable_Load.brd (EAGLE design)
At the start: 125.7 x 41.9 mm, 52 parts, among them Q1 60V/32A/35mΩ, U1 CY8C5868LTI-LP039, U2 3.3V

Commit message: Removed header for CT keypad
Parts:
- removed J1: (no value), SparkFun-Connectors:1X05
Connections:
- removed net KP_IRQ: J1.2, U1.2
- removed net SCL: J1.3, U1.68
- removed net SDA: J1.4, U1.1
- net 3.3V: no longer J1.1
- net GND: no longer J1.5
Routing:
- net SDA: track 22.8 -> 0.00 mm, vias 1 -> 0
- net SCL: track 20.5 -> 0.00 mm, vias 2 -> 0
- net KP_IRQ: track 19.5 -> 0.00 mm, vias 1 -> 0
- net 3.3V: track 34.9 -> 27.8 mm
Other:
- board text removed: "3.3V"
- board text removed: "IRQ"
- board text removed: "SCL"
- board text removed: "SDA"
Changed lines of the file:
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@@
 <text x="6.604" y="26.035" size="1.27" layer="21" font="vector" ratio="15">RXI</text>
 <text x="6.604" y="23.495" size="1.27" layer="21" font="vector" ratio="15">TXO</text>
-<text x="2.794" y="19.685" size="1.27" layer="21" font="vector" ratio="15">GND</text>
-<text x="2.794" y="17.145" size="1.27" layer="21" font="vector" ratio="15">SDA</text>
-<text x="2.794" y="14.605" size="1.27" layer="21" font="vector" ratio="15">SCL</text>
-<text x="2.794" y="12.065" size="1.27" layer="21" font="vector" ratio="15">IRQ</text>
-<text x="2.794" y="9.525" size="1.27" layer="21" font="vector" ratio="15">3.3V</text>
 <text x="62.738" y="30.607" size="1.27" layer="21" font="vector" ratio="15" rot="R90">LOAD_GND</text>
 <text x="66.548" y="30.607" size="1.27" layer="21" font="vector" ratio="15" rot="R90">LOAD_POS</text>
@@
 <attribute name="PROD_ID" value="COMP-09537" x="91.44" y="28.575" size="1.778" layer="28" rot="MR180" display="off"/>
 </element>
-<element name="J1" library="SparkFun-Connectors" package="1X05" value="" x="1.27" y="10.16" rot="R90"/>
 <element name="J2" library="SparkFun-Connectors" package="1X16" value="" x="115.57" y="1.27" rot="MR0"/>
 <element name="J3" library="SparkFun-Connectors" package="USB-MICROB" value="" x="19.05" y="40.64" rot="R90">
@@
 <contactref element="U1" pad="45"/>
 <contactref element="U1" pad="25"/>
-<contactref element="J1" pad="5"/>
 <contactref element="J2" pad="1"/>
 <contactref element="J2" pad="3"/>
@@
 <signal name="3.3V">
 <contactref element="U1" pad="67"/>
-<contactref element="J1" pad="1"/>
 <contactref element="U2" pad="5"/>
 <contactref element="C5" pad="1"/>
@@
 <wire x1="8.763" y1="15.367" x2="8.763" y2="10.541" width="0.4064" layer="15"/>
 <wire x1="8.763" y1="10.541" x2="8.382" y2="10.16" width="0.4064" layer="15"/>
-<wire x1="8.382" y1="10.16" x2="1.27" y2="10.16" width="0.4064" layer="15"/>
 </signal>
 <signal name="5V">
@@
 <wire x1="105.41" y1="4.318" x2="105.41" y2="1.27" width="0.2032" layer="16"/>
 </signal>
-<signal name="SCL">
-<contactref element="U1" pad="68"/>
-<contactref element="J1" pad="3"/>
-<wire x1="16.42" y1="15.85" x2="15.723" y2="15.85" width="0.2032" layer="1"/>
-<wire x1="15.723" y1="15.85" x2="15.621" y2="15.748" width="0.2032" layer="1"/>
-<wire x1="15.621" y1="15.748" x2="15.621" y2="12.827" width="0.2032" layer="1"/>
-<wire x1="15.621" y1="12.827" x2="15.494" y2="12.7" width="0.2032" layer="1"/>
-<wire x1="15.494" y1="12.7" x2="10.033" y2="12.7" width="0.2032" layer="1"/>
-<via x="10.033" y="12.7" extent="1-16" drill="0.254"/>
-<wire x1="10.033" y1="12.7" x2="7.62" y2="12.7" width="0.2032" layer="16"/>
-<via x="7.62" y="12.7" extent="1-16" drill="0.254"/>
-<wire x1="7.62" y1="12.7" x2="7.62" y2="14.859" width="0.2032" layer="1"/>
-<wire x1="7.62" y1="14.859" x2="7.239" y2="15.24" width="0.2032" layer="1"/>
-<wire x1="7.239" y1="15.24" x2="1.27" y2="15.24" width="0.2032" layer="1"/>
-</signal>
-<signal name="SDA">
-<contactref element="U1" pad="1"/>
-<contactref element="J1" pad="4"/>
-<wire x1="17.12" y1="15.15" x2="17.12" y2="14.707" width="0.2032" layer="1"/>
-<wire x1="17.12" y1="14.707" x2="16.764" y2="14.351" width="0.2032" layer="1"/>
-<wire x1="16.764" y1="14.351" x2="16.51" y2="14.351" width="0.2032" layer="1"/>
-<wire x1="16.51" y1="14.351" x2="16.129" y2="13.97" width="0.2032" layer="1"/>
-<wire x1="16.129" y1="13.97" x2="16.129" y2="12.7" width="0.2032" layer="1"/>
-<wire x1="16.129" y1="12.7" x2="15.748" y2="12.319" width="0.2032" layer="1"/>
-<wire x1="15.748" y1="12.319" x2="10.414" y2="12.319" width="0.2032" layer="1"/>
-<wire x1="10.414" y1="12.319" x2="10.033" y2="11.938" width="0.2032" layer="1"/>
-<via x="10.033" y="11.938" extent="1-16" drill="0.254"/>
-<wire x1="10.033" y1="11.938" x2="3.302" y2="11.938" width="0.2032" layer="16"/>
-<wire x1="3.302" y1="11.938" x2="2.54" y2="12.7" width="0.2032" layer="16"/>
-<wire x1="2.54" y1="12.7" x2="2.54" y2="16.51" width="0.2032" layer="16"/>
-<wire x1="2.54" y1="16.51" x2="1.27" y2="17.78" width="0.2032" layer="16"/>
-</signal>
-<signal name="KP_IRQ">
-<contactref element="U1" pad="2"/>
-<contactref element="J1" pad="2"/>
-<wire x1="17.52" y1="15.15" x2="17.52" y2="14.599" width="0.2032" layer="1"/>
-<wire x1="17.52" y1="14.599" x2="16.51" y2="13.589" width="0.2032" layer="1"/>
-<wire x1="16.51" y1="13.589" x2="16.51" y2="12.446" width="0.2032" layer="1"/>
-<wire x1="16.51" y1="12.446" x2="16.002" y2="11.938" width="0.2032" layer="1"/>
-<wire x1="16.002" y1="11.938" x2="10.795" y2="11.938" width="0.2032" layer="1"/>
-<wire x1="10.795" y1="11.938" x2="10.033" y2="11.176" width="0.2032" layer="1"/>
-<via x="10.033" y="11.176" extent="1-16" drill="0.254"/>
-<wire x1="10.033" y1="11.176" x2="2.794" y2="11.176" width="0.2032" layer="16"/>
-<wire x1="2.794" y1="11.176" x2="1.27" y2="12.7" width="0.2032" layer="16"/>
-</signal>
 <signal name="N$6">
